Commit message: control

File: public/tu_nguyen/urdf/tu_nguyen.urdf (robot description, URDF)
Before this commit: robot tu_nguyen, 7 links, 6 joints
Joints:
- joint joint_2: origin xyz=0.00010548 -0.024031 0.044 rpy=0 0 0 -> xyz=0.00010548 -0.024031 0.044 rpy=0 0.3 0
- joint joint_3: origin xyz=0 0 0.12194 rpy=0 0 0 -> xyz=0 0 0.12194 rpy=0 0.8 0
- joint joint_4: origin xyz=0 0 0.114 rpy=0 0 0 -> xyz=0 0 0.114 rpy=0 0.5 0
